Commit message: wip

File: src/my_robot/urdf/my_robot.xacro (robot description, xacro)
@@ -1,5 +1,12 @@
 <?xml version='1.0'?>
 <robot name="my_robot" xmlns:xacro="http://www.ros.org/wiki/xacro">
+    <xacro:include filename="$(find my_robot)/urdf/my_robot.gazebo" />
     <link name="robot_footprint"></link>
+    <gazebo reference="left_wheel">
+        <material>Gazebo/Green</material>
+    </gazebo>
+    <gazebo reference="right_wheel">
+        <material>Gazebo/Green</material>
+    </gazebo>
     <joint name="robot_footprint_joint" type="fixed">
         <origin xyz="0 0 0" rpy="0 0 0"/>
@@ -22,4 +29,16 @@
         <limit effort="10000" velocity="1000"/>
         <dynamics damping="1.0" friction="1.0"/>
+    </joint>
+    <joint type="fixed" name="camera_joint">
+        <origin xyz="0.2 0 0" rpy="0 0 0"/>
+        <child link="camera"/>
+        <parent link="chassis"/>
+        <axis xyz="0 1 0" rpy="0 0 0"/>
+    </joint>
+    <joint type="fixed" name="hokuyo_joint">
+        <origin xyz="0.15 0 .1" rpy="0 0 0"/>
+        <child link="hokuyo"/>
+        <parent link="chassis"/>
+        <axis xyz="0 1 0" rpy="0 0 0"/>
     </joint>
     <link name='chassis'>
@@ -72,5 +91,4 @@
     </link>
     <link name='left_wheel'>
-        <pose>0 0 0.1 0 0 0</pose>
         <inertial>
             <mass value="5.0"/>
@@ -96,5 +114,4 @@
     </link>
     <link name='right_wheel'>
-        <pose>0 0 0.1 0 0 0</pose>
         <inertial>
             <mass value="5.0"/>
@@ -119,3 +136,49 @@
         </visual>
     </link>
+    <link name='camera'>
+        <inertial>
+            <mass value="0.1"/>
+            <origin xyz="0.0 0 0" rpy="0 0 0"/>
+            <inertia
+                    ixx="1e-6" ixy="0" ixz="0"
+                    iyy="1e-6" iyz="0"
+                    izz="1e-6"
+            />
+        </inertial>
+        <collision>
+            <origin xyz="0 0 0" rpy="0 0 0"/>
+            <geometry>
+                <box size="0.05 0.05 0.05"/>
+            </geometry>
+        </collision>
+        <visual>
+            <origin xyz="0 0 0" rpy="0 0 0"/>
+            <geometry>
+                <box size="0.05 0.05 0.05"/>
+            </geometry>
+        </visual>
+    </link>
+    <link name="hokuyo">
+        <inertial>
+            <mass value="1e-5"/>
+            <origin xyz="0 0 0" rpy="0 0 0"/>
+            <inertia
+                    ixx="1e-6" ixy="0.0" ixz="0.0"
+                    iyy="1e-6" iyz="0.0"
+                    izz="1e-6"
+            />
+        </inertial>
+        <collision>
+            <origin xyz="0 0 0" rpy="0 0 0"/>
+            <geometry>
+                <box size="0.1 0.1 0.1"/>
+            </geometry>
+        </collision>
+        <visual>
+            <origin xyz="0 0 0" rpy="0 0 0"/>
+            <geometry>
+                <mesh filename="package://my_robot/meshes/hokuyo.dae"/>
+            </geometry>
+        </visual>
+    </link>
 </robot>
